File: TCE.kicad_pcb (KiCad board)
At the start: 2 copper layers, 50 x 128.5 mm, 58 parts, among them J1 rca, J2 rca, J3 europower, Q1 2N3904, SW1 SW_DPDT_x2, U1 LM339, U2 LM317, U3 L78L05

Commit message: .gitignore, image of pcb/panel, shift C3 slightly
Parts:
- moved C3 2.25 mm to (1.68, 57.2)
Routing:
- net VIDEO_IN: track 51.4 -> 53.6 mm
Changed lines of the file:
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@@
       (effects (font (size 1 1) (thickness 0.15)))
     )
-    (fp_text value "LM339" (at 3.81 17.57 90) (layer "F.Fab")
+    (fp_text value "LM339" (at 3.79 15.455 90) (layer "F.Fab")
       (effects (font (size 1 1) (thickness 0.15)))
     )
@@
   )
   (footprint "Capacitor_THT:C_Disc_D4.7mm_W2.5mm_P5.00mm" (layer "F.Cu")
-    (at 1.725 54.975 -90)
+    (at 1.675 57.225 -90)
     (descr "C, Disc series, Radial, pin pitch=5.00mm, , diameter*width=4.7*2.5mm^2, Capacitor, http://www.vishay.com/docs/45233/krseries.pdf")
     (tags "C Disc series Radial pin pitch 5.00mm  diameter 4.7mm width 2.5mm Capacitor")
@@
     (property "Sheetname" "User Interface")
     (attr through_hole)
-    (fp_text reference "C3" (at 4.125 -2.175 -90) (layer "F.SilkS")
+    (fp_text reference "C3" (at 2.75 -2.225 -90) (layer "F.SilkS")
       (effects (font (size 1 1) (thickness 0.15)))
     )
@@
     (property "Sheetname" "User Interface")
     (attr through_hole)
-    (fp_text reference "D1" (at 3.335 -0.375 90) (layer "F.SilkS")
+    (fp_text reference "D1" (at -1.865 -0.025 180) (layer "F.SilkS")
       (effects (font (size 1 1) (thickness 0.15)))
     )
@@
       (effects (font (size 1 1) (thickness 0.15)))
     )
-    (fp_text value "0.1u" (at 2.5 2.5 90) (layer "F.Fab")
+    (fp_text value "0.1u" (at 2.725 0.65 90) (layer "F.Fab")
       (effects (font (size 1 1) (thickness 0.15)))
     )
-    (fp_text user "${REFERENCE}" (at 2.5 0 90) (layer "F.Fab")
+    (fp_text user "${REFERENCE}" (at 1.75 -0.55 90) (layer "F.Fab")
       (effects (font (size 0.94 0.94) (thickness 0.141)))
     )
@@
       (effects (font (size 1 1) (thickness 0.15)))
     )
-    (fp_text value "1u" (at 2.5 2.5 90) (layer "F.Fab")
+    (fp_text value "1u" (at 1.855 0.555 90) (layer "F.Fab")
       (effects (font (size 1 1) (thickness 0.15)))
     )
-    (fp_text user "${REFERENCE}" (at 2.5 0 90) (layer "F.Fab")
+    (fp_text user "${REFERENCE}" (at 3.255 -0.645 90) (layer "F.Fab")
       (effects (font (size 0.94 0.94) (thickness 0.141)))
     )
@@
     (property "Sheetname" "Power")
     (attr through_hole)
-    (fp_text reference "D3" (at 6.31 -2.175 90) (layer "B.SilkS")
+    (fp_text reference "D3" (at 5.46 2.325 90) (layer "B.SilkS")
       (effects (font (size 1 1) (thickness 0.15)) (justify mirror))
     )
-    (fp_text value "1n4007" (at 3.885 -2.225 90) (layer "B.Fab")
+    (fp_text value "1n4007" (at 3.91 0 90) (layer "B.Fab")
       (effects (font (size 1 1) (thickness 0.15)) (justify mirror))
     )
@@
   (segment (start 4.955 17.735) (end 4.955 9.545) (width 0.25) (layer "B.Cu") (net 3))
   (segment (start 5 53.1) (end 2.19 53.1) (width 0.25) (layer "F.Cu") (net 4))
+  (segment (start 1.7 52.61) (end 1.7 57.2) (width 0.25) (layer "F.Cu") (net 4))
   (segment (start 2.19 53.1) (end 1.7 52.61) (width 0.25) (layer "F.Cu") (net 4))
-  (segment (start 1.725 54.975) (end 1.725 52.635) (width 0.25) (layer "F.Cu") (net 4))
-  (segment (start 1.725 52.635) (end 1.7 52.61) (width 0.25) (layer "F.Cu") (net 4))
+  (segment (start 1.675 52.635) (end 1.7 52.61) (width 0.25) (layer "F.Cu") (net 4))
   (segment (start 7.495 17.735) (end 7.495 22.815) (width 0.25) (layer "F.Cu") (net 4))
   (segment (start 7.495 22.815) (end 10.035 25.355) (width 0.25) (layer "F.Cu") (net 4))
   (segment (start 2.415 17.735) (end 3.94 16.21) (width 0.25) (layer "F.Cu") (net 4))
+  (segment (start 1.7 57.2) (end 1.675 57.225) (width 0.25) (layer "F.Cu") (net 4))
   (segment (start 5.97 16.21) (end 7.495 17.735) (width 0.25) (layer "F.Cu") (net 4))
   (segment (start 3.94 16.21) (end 5.97 16.21) (width 0.25) (layer "F.Cu") (net 4))
@@
   (segment (start 5 53.1) (end 6.675 51.425) (width 0.25) (layer "B.Cu") (net 4))
   (segment (start 6.675 41.166444) (end 5.903557 40.395001) (width 0.25) (layer "B.Cu") (net 4))
-  (segment (start 1.725 59.975) (end 7.375 65.625) (width 0.25) (layer "F.Cu") (net 5))
-  (segment (start 7.375 65.625) (end 7.6 65.625) (width 0.25) (layer "F.Cu") (net 5))
-  (segment (start 8.15863 52.41) (end 9.525 52.41) (width 0.25) (layer "F.Cu") (net 5))
-  (segment (start 1.725 59.975) (end 1.725 58.84363) (width 0.25) (layer "F.Cu") (net 5))
-  (segment (start 1.725 58.84363) (end 8.15863 52.41) (width 0.25) (layer "F.Cu") (net 5))
+  (segment (start 9.525 52.41) (end 8.39363 52.41) (width 0.25) (layer "F.Cu") (net 5))
+  (segment (start 1.675 62.225) (end 4.2 62.225) (width 0.25) (layer "F.Cu") (net 5))
+  (segment (start 8.39363 52.41) (end 4.2 56.60363) (width 0.25) (layer "F.Cu") (net 5))
+  (segment (start 4.2 62.225) (end 7.6 65.625) (width 0.25) (layer "F.Cu") (net 5))
+  (segment (start 4.2 56.60363) (end 4.2 62.225) (width 0.25) (layer "F.Cu") (net 5))
   (segment (start 18.64 42.21) (end 14.23 37.8) (width 0.25) (layer "F.Cu") (net 6))
   (segment (start 18.35 6.425) (end 18.35 8.875) (width 0.25) (layer "F.Cu") (net 6))

Commit message: 2nd 3D rendering, changes to silkscreen text
Parts:
- moved Ref** 0.80 mm to (10.0, 102.0)
Other:
- board text added: "eurorack version by bfisher/octovolt"
- board text removed: "eurorack version by octopus-arts"
Changed lines of the file:
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@@
   )
   (footprint "Graphics:octopus_silk_screen" (layer "B.Cu")
-    (at 10.009903 102.804887 180)
+    (at 10 102 180)
     (attr through_hole exclude_from_bom)
     (fp_text reference "Ref**" (at 0 0) (layer "B.SilkS") hide
@@
     (fp_line (start 4.83 -6.62) (end 3.34 -6.62) (layer "B.SilkS") (width 0.12))
     (fp_line (start 4.83 -6.62) (end 4.83 -1.9) (layer "B.SilkS") (width 0.12))
-    (fp_line (start 4.83 1.91) (end 4.83 4.97) (layer "B.SilkS") (width 0.12))
     (fp_line (start -4.92 -6.62) (end -4.92 -1.9) (layer "B.SilkS") (width 0.12))
     (fp_line (start -0.83 -6.62) (end -1.36 -6.62) (layer "B.SilkS") (width 0.12))
     (fp_line (start 4.83 4.97) (end -4.91 4.97) (layer "B.SilkS") (width 0.12))
-    (fp_line (start -4.91 1.91) (end -4.91 4.97) (layer "B.SilkS") (width 0.12))
     (fp_circle (center 0 0) (end 6.357366 0) (layer "B.SilkS") (width 0.15) (fill none))
     (fp_line (start 6.37 -8.65) (end 6.37 5.1) (layer "B.CrtYd") (width 0.05))
@@
     (effects (font (size 1 1) (thickness 0.15)) (justify mirror))
   )
-  (gr_text "JCLJCLJCLJCL" (at 15.6 46.3 90) (layer "B.SilkS")
+  (gr_text "JCLJCLJCLJCL" (at 9.975 2.775) (layer "B.SilkS")
     (effects (font (size 1 1) (thickness 0.15)) (justify mirror))
   )
-  (gr_text "TCE: Two Comparator Effect v.0.1.3" (at 10 19.66) (layer "B.SilkS")
+  (gr_text "TCE: Two Comparator Effect v.0.1.3" (at 10 20.45) (layer "B.SilkS")
     (effects (font (size 0.7 0.7) (thickness 0.12)) (justify mirror))
   )
@@
     (effects (font (size 1 1) (thickness 0.15)) (justify mirror))
   )
-  (gr_text "adapted from a rob schafer design" (at 10 20.56) (layer "B.SilkS")
+  (gr_text "adapted from a rob schafer design" (at 10 47.525) (layer "B.SilkS")
     (effects (font (size 0.7 0.7) (thickness 0.12)) (justify mirror))
   )
@@
     (effects (font (size 1 1) (thickness 0.15)) (justify mirror))
   )
-  (gr_text "GNU General Public License v3.0" (at 10 23.52) (layer "B.SilkS")
+  (gr_text "GNU General Public License v3.0" (at 10 104.95) (layer "B.SilkS")
     (effects (font (size 0.7 0.7) (thickness 0.12)) (justify mirror))
   )
-  (gr_text "eurorack version by octopus-arts" (at 9.75 22.36) (layer "B.SilkS")
+  (gr_text "eurorack version by bfisher/octovolt" (at 10.075 50.275) (layer "B.SilkS")
     (effects (font (size 0.7 0.7) (thickness 0.12)) (justify mirror))
   )
@@
     (effects (font (size 1 1) (thickness 0.15)) (justify mirror))
   )
-  (gr_text "by cyberboy666" (at 10 21.46) (layer "B.SilkS")
+  (gr_text "by cyberboy666" (at 10.05 48.81) (layer "B.SilkS")
     (effects (font (size 0.7 0.7) (thickness 0.12)) (justify mirror))
   )
